File: Projects/AKK/BLDC_Motor_Controller/Design/rev01/rev01_1/Motor_Controller/Motor_Controller.kicad_sch (KiCad schematic)
At the start: 0 parts

Commit message: Update_02
Created project and MCU schematic.
Other:
- added sheet [01] BLOCK DIAGRAM ([01] BLOCK DIAGRAM.kicad_sch)
- added sheet [02] INPUT PROTECTION ([02] INPUT PROTECTION.kicad_sch)
- added sheet [03] STEP DOWN ([03] STEP DOWN.kicad_sch)
- added sheet [04] MCU ([04] MCU.kicad_sch)
- added sheet [05] MOSFET DRIVER ([05] MOSFET DRIVER.kicad_sch)
- added sheet [06] MOSFETS ([06] MOSFETS.kicad_sch)
- added sheet [07] CAN ([07] CAN.kicad_sch)
- added sheet [08] FILTERS ([08] FILTERS.kicad_sch)
- added sheet [09] USB ([09] USB.kicad_sch)
- added sheet [10] MECHANICAL ([10] MECHANICAL.kicad_sch)
- note added: "1"
- note added: "10"
- note added: "2"
- note added: "3"
- note added: "4"
- note added: "5"
- note added: "6"
- note added: "7"
- note added: "8"
- note added: "9"
- note added: "BACK VIEW"
- note added: "BLOCK DIAGRAM"
- note added: "CAN"
- note added: "DATE: ${ISSUE_DATE}"
- note added: "DRAFT"
- note added: "FILTERS"
- note added: "FRONT VIEW"
- note added: "INDEX"
- note added: "INPUT PROTECTION"
- note added: "MCU"
- note added: "MECHANICAL"
- note added: "MOSFET DRIVER"
- note added: "MOSFETs"
- note added: "Motor_Controller"
- note added: "PAGE"
- note added: "REALEASE STATUS PROJECT:"
- note added: "REVISIONS: 01_1"
- note added: "STEP DOWN"
- note added: "USB"
- note added: "VARIANTS: NO VARIANT"

Commit message: Update_03
Completed schematic.
Changed lines of the file:
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@@
 		(at 146.05 67.31)
 		(size 22.86 17.78)
-		(fields_autoplaced yes)
 		(stroke
 			(width 1)
@@
 			)
 		)
-		(instances
-			(project "Motor_Controller"
-				(path "/e63e39d7-6ac0-4ffd-8aa3-1841a4541b55"
-					(page "5")
+		(property "Pagenumber" "4"
+			(at 167.386 83.312 0)
+			(effects
+				(font
+					(size 3 3)
+					(bold yes)
+					(color 0 0 255 1)
+				)
+				(justify right bottom)
+			)
+		)
+		(instances
+			(project "Motor_Controller"
+				(path "/e63e39d7-6ac0-4ffd-8aa3-1841a4541b55"
+					(page "04")
 				)
 			)
@@
 		(at 146.05 34.29)
 		(size 22.86 17.78)
-		(fields_autoplaced yes)
 		(stroke
 			(width 1)
@@
 			)
 		)
-		(instances
-			(project "Motor_Controller"
-				(path "/e63e39d7-6ac0-4ffd-8aa3-1841a4541b55"
-					(page "3")
+		(property "Pagenumber" "2"
+			(at 167.386 50.292 0)
+			(effects
+				(font
+					(size 3 3)
+					(bold yes)
+					(color 0 0 255 1)
+				)
+				(justify right bottom)
+			)
+		)
+		(instances
+			(project "Motor_Controller"
+				(path "/e63e39d7-6ac0-4ffd-8aa3-1841a4541b55"
+					(page "02")
 				)
 			)
@@
 		(at 109.22 67.31)
 		(size 22.86 17.78)
-		(fields_autoplaced yes)
 		(stroke
 			(width 1)
@@
 			)
 		)
-		(instances
-			(project "Motor_Controller"
-				(path "/e63e39d7-6ac0-4ffd-8aa3-1841a4541b55"
-					(page "4")
+		(property "Pagenumber" "3"
+			(at 130.302 83.058 0)
+			(effects
+				(font
+					(size 3 3)
+					(bold yes)
+					(color 0 0 255 1)
+				)
+				(justify right bottom)
+			)
+		)
+		(instances
+			(project "Motor_Controller"
+				(path "/e63e39d7-6ac0-4ffd-8aa3-1841a4541b55"
+					(page "03")
 				)
 			)
@@
 		(at 109.22 34.29)
 		(size 22.86 17.78)
-		(fields_autoplaced yes)
 		(stroke
 			(width 1)
@@
 			)
 		)
-		(instances
-			(project "Motor_Controller"
-				(path "/e63e39d7-6ac0-4ffd-8aa3-1841a4541b55"
-					(page "2")
+		(property "Pagenumber" "1"
+			(at 130.81 50.546 0)
+			(effects
+				(font
+					(size 3 3)
+					(bold yes)
+					(color 0 0 255 1)
+				)
+				(justify right bottom)
+			)
+		)
+		(instances
+			(project "Motor_Controller"
+				(path "/e63e39d7-6ac0-4ffd-8aa3-1841a4541b55"
+					(page "01")
 				)
 			)
@@
 		(at 222.25 67.31)
 		(size 22.86 17.78)
-		(fields_autoplaced yes)
 		(stroke
 			(width 1)
@@
 			)
 		)
-		(instances
-			(project "Motor_Controller"
-				(path "/e63e39d7-6ac0-4ffd-8aa3-1841a4541b55"
-					(page "7")
+		(property "Pagenumber" "6"
+			(at 242.824 82.55 0)
+			(effects
+				(font
+					(size 3 3)
+					(bold yes)
+					(color 0 0 255 1)
+				)
+				(justify right bottom)
+			)
+		)
+		(instances
+			(project "Motor_Controller"
+				(path "/e63e39d7-6ac0-4ffd-8aa3-1841a4541b55"
+					(page "06")
 				)
 			)
@@
 		(at 109.22 101.6)
 		(size 22.86 17.78)
-		(fields_autoplaced yes)
 		(stroke
 			(width 1)
@@
 			)
 		)
-		(instances
-			(project "Motor_Controller"
-				(path "/e63e39d7-6ac0-4ffd-8aa3-1841a4541b55"
-					(page "8")
+		(property "Pagenumber" "7"
+			(at 129.794 117.094 0)
+			(effects
+				(font
+					(size 3 3)
+					(bold yes)
+					(color 0 0 255 1)
+				)
+				(justify right bottom)
+			)
+		)
+		(instances
+			(project "Motor_Controller"
+				(path "/e63e39d7-6ac0-4ffd-8aa3-1841a4541b55"
+					(page "07")
 				)
 			)
@@
 		(at 182.88 67.31)
 		(size 22.86 17.78)
-		(fields_autoplaced yes)
 		(stroke
 			(width 1)
@@
 			)
 		)
-		(instances
-			(project "Motor_Controller"
-				(path "/e63e39d7-6ac0-4ffd-8aa3-1841a4541b55"
-					(page "6")
+		(property "Pagenumber" "5"
+			(at 204.216 83.058 0)
+			(effects
+				(font
+					(size 3 3)
+					(bold yes)
+					(color 0 0 255 1)
+				)
+				(justify right bottom)
+			)
+		)
+		(instances
+			(project "Motor_Controller"
+				(path "/e63e39d7-6ac0-4ffd-8aa3-1841a4541b55"
+					(page "05")
 				)
 			)
@@
 		(at 182.88 101.6)
 		(size 22.86 17.78)
-		(fields_autoplaced yes)
 		(stroke
 			(width 1)
@@
 		)
 		(property "Sheetname" "[09] USB"
-			(at 182.88 100.8884 0)
+			(at 182.88 100.4646 0)
 			(effects
 				(font
@@
 		)
 		(property "Sheetfile" "[09] USB.kicad_sch"
-			(at 182.88 119.9646 0)
-			(effects
-				(font
-					(size 1.27 1.27)
-				)
-				(justify left top)
+			(at 182.88 120.3884 0)
+			(effects
+				(font
+					(size 1.27 1.27)
+				)
+				(justify left top)
+			)
+		)
+		(property "Pagenumber" "9"
+			(at 204.47 117.856 0)
+			(effects
+				(font
+					(size 3 3)
+					(bold yes)
+					(color 0 0 255 1)
+				)
+				(justify right bottom)
+			)
+		)
+		(instances
+			(project "Motor_Controller"
+				(path "/e63e39d7-6ac0-4ffd-8aa3-1841a4541b55"
+					(page "09")
+				)
+			)
+		)
+	)
+	(sheet
+		(at 222.25 101.6)
+		(size 22.86 17.78)
+		(stroke
+			(width 1)
+			(type solid)
+		)
+		(fill
+			(color 31 169 39 1.0000)
+		)
+		(property "Sheetname" "[10] MECHANICAL"
+			(at 222.25 100.4646 0)
+			(effects
+				(font
+					(size 1.27 1.27)
+				)
+				(justify left bottom)
+			)
+		)
+		(property "Sheetfile" "[10] MECHANICAL.kicad_sch"
+			(at 222.25 120.3884 0)
+			(effects
+				(font
+					(size 1.27 1.27)
+				)
+				(justify left top)
+			)
+		)
+		(property "Pagenumber" "10"
+			(at 243.586 117.856 0)
+			(effects
+				(font
+					(size 3 3)
+					(bold yes)
+					(color 0 0 255 1)
+				)
+				(justify right bottom)
 			)
 		)
@@
 	)
 	(sheet
-		(at 222.25 101.6)
-		(size 22.86 17.78)
-		(fields_autoplaced yes)
-		(stroke
-			(width 1)
-			(type solid)
-		)
-		(fill
-			(color 31 169 39 1.0000)
-		)
-		(property "Sheetname" "[10] MECHANICAL"
-			(at 222.25 100.8884 0)
-			(effects
-				(font
-					(size 1.27 1.27)
-				)
-				(justify left bottom)
-			)
-		)
-		(property "Sheetfile" "[10] MECHANICAL.kicad_sch"
-			(at 222.25 119.9646 0)
-			(effects
-				(font
-					(size 1.27 1.27)
-				)
-				(justify left top)
-			)
-		)
-		(instances
-			(project "Motor_Controller"
-				(path "/e63e39d7-6ac0-4ffd-8aa3-1841a4541b55"
-					(page "11")
-				)
-			)
-		)
-	)
-	(sheet
 		(at 146.05 101.6)
 		(size 22.86 17.78)
-		(fields_autoplaced yes)
 		(stroke
 			(width 1)
@@
 		)
 		(property "Sheetname" "[08] FILTERS"
-			(at 146.05 100.8884 0)
+			(at 146.05 100.4646 0)
 			(effects
 				(font
@@
 		)
 		(property "Sheetfile" "[08] FILTERS.kicad_sch"
-			(at 146.05 119.9646 0)
-			(effects
-				(font
-					(size 1.27 1.27)
-				)
-				(justify left top)
-			)
-		)
-		(instances
-			(project "Motor_Controller"
-				(path "/e63e39d7-6ac0-4ffd-8aa3-1841a4541b55"
-					(page "9")
-				)
-			)
+			(at 146.05 120.3884 0)
+			(effects
+				(font
+					(size 1.27 1.27)
+				)
+				(justify left top)
+			)
+		)
+		(property "Pagenumber" "8"
+			(at 167.132 117.856 0)
+			(effects
+				(font
+					(size 3 3)
+					(bold yes)
+					(color 0 0 255 1)
+				)
+				(justify right bottom)
+			)
+		)
+		(instances
+			(project "Motor_Controller"
+				(path "/e63e39d7-6ac0-4ffd-8aa3-1841a4541b55"
+					(page "08")
+				)
+			)
