File: Projects/AKK/BLDC_Motor_Controller/Design/rev01/rev01_1/Motor_Controller/[03] STEP DOWN.kicad_sch (KiCad schematic)
At the start: 0 parts

Commit message: Update_03
Completed schematic.
Parts:
- added C44, C45, C46, C47: 1u, symbol Device:C
- added D12, D14: LED_G, symbol Device:LED
- added D13: BAT60A, Diode_SMD:D_SOD-323, symbol Diode:BAT60A
- added R24, R25: 1k, symbol Device:R
- added U4: AMS1117-3.3, Package_TO_SOT_SMD:SOT-223-3_TabPin2, symbol Regulator_Linear:AMS1117-3.3
Connections:
- new net: D12.2 (A), R24.2
- new net: D14.2 (A), R25.2
- new net +3V3: D13.1 (K), R25.1
- new net +3V3_IC: C46.1, C47.1, D13.2 (A), U4.2 (VO)
- new net +5V: C44.1, C45.1, R24.1, U4.3 (VI)
- new net GND: C44.2, C45.2, C46.2, C47.2, D12.1 (K), D14.1 (K), U4.1 (GND)
Other:
- note added: "FROM MOSFET DRIVER OR EXTERNAL"
- note added: "[03] STEP DOWN"
