File: Projects/AKK/BLDC_Motor_Controller/Design/rev01/rev01_1/Motor_Controller/[04] MCU.kicad_sch (KiCad schematic)
At the start: 36 parts, among them J1 Conn_01x08, J2 Conn_01x06, J3 Conn_01x03, SW1 SW_DIP_x01, U1 STM32F405RGTx, Y1 Crystal

Commit message: Update_03
Completed schematic.
Changed lines of the file:
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@@
 	)
 	(rectangle
-		(start 230.124 13.462)
+		(start 229.87 13.462)
 		(end 279.654 84.074)
 		(stroke
@@
 	(text "[04] MCU"
 		(exclude_from_sim no)
-		(at 148.082 19.812 0)
+		(at 136.144 18.542 0)
 		(effects
 			(font
