File: Projects/AKK/BLDC_Motor_Controller/Design/rev01/rev01_1/Motor_Controller/[05] MOSFET DRIVER.kicad_sch (KiCad schematic)
At the start: 0 parts

Commit message: Update_03
Completed schematic.
Parts:
- added C16: 10n, symbol Device:C
- added C17: 120p, symbol Device:C
- added C18, C19, C20, C22, C23: 2u2, symbol Device:C
- added C21: 22n, symbol Device:C
- added C24, C25, C26, C27, C28, C29, C30: 100n, symbol Device:C
- added C31, C32, C33: 10u, symbol Device:C
- added C34, C35, C36, C37, C38, C39: 1u, symbol Device:C
- added D8: PMEG6020, Diode_SMD:Nexperia_CFP3_SOD-123W, symbol Diode:PMEG6020ER
- added D9: BAT60A, Diode_SMD:D_SOD-323, symbol Diode:BAT60A
- added L1: 22u, symbol Device:L
- added NT1: NetTie_2, symbol Device:NetTie_2
- added R10: 10k, symbol Device:R
- added R11: 1M, symbol Device:R
- added R12: 18k, symbol Device:R
- added R13: 3k3, symbol Device:R
- added R14, R16, R18: 39k, symbol Device:R
- added R15, R17, R19: 2k2, symbol Device:R
- added R8: 16k, symbol Device:R
- added R9: 205k, symbol Device:R
- added U2: DRV8302DCAR, DRV8302_footprint_lib:HTSSOP-56_L14.0-W6.1-P0.50-LS8.1-BL-EP, symbol DRV8302:DRV8302DCAR
Connections:
- new net: C20.1, C22.1, U2.13 (GVDD)
- new net: C23.1, U2.27 (AVDD)
- new net: C16.2, R8.2
- new net: C30.1, U2.52 (BST_BK)
- new net: C21.1, U2.14 (CP1)
- new net: C21.2, U2.15 (CP2)
- new net +3V3: U2.24 (REF), U2.9 (M_OC)
- new net +5V: D9.1 (K)
- new net +5V_DRV: C31.1, C32.1, C33.1, D9.2 (A), L1.2, R12.2
- new net +VDC: C24.1, C25.1, C26.1, C34.1, C35.1, C36.1, C37.1, C38.1, C39.1, U2.29 (PVDD1), U2.53 (PVDD2), U2.54 (PVDD2)
- new net BIAS: R11.1, U2.49 (BIAS)
- new net BR_SO1: U2.25 (SO1)
- new net BR_SO2: U2.26 (SO2)
- new net BST_A: C27.1, U2.48 (BST_A)
- new net BST_B: C28.1, U2.43 (BST_B)
- new net BST_C: C29.1, U2.38 (BST_C)
- new net COMP: C17.2, R8.1, U2.2 (COMP)
- new net DC_CAL: U2.12 (DC_CAL)
- new net DTC: R10.2, U2.7 (DTC)
- new net DVDD: NT1.1, U2.23 (DVDD)
- new net EN_GATE: U2.16 (EN_GATE)
- new net FAULT: U2.6 (nFAULT)
- new net GND: C16.1, C17.1, C18.2, C19.2, C20.2, C22.2, C23.2, C24.2, C25.2, C26.2, C31.2, C32.2, C33.2, C34.2, C35.2, C36.2, C37.2, C38.2, C39.2, D8.2 (A), R10.1, R11.2, R13.1, R15.1, R17.1, R19.1, R9.1, U2.10 (GAIN), U2.28 (AGND), U2.57 (GND), U2.8 (M_PWM)
- new net H1: U2.17 (INH_A)
- new net H1_LOW: U2.44 (SL_A)
- new net H1_VS: C27.2, R18.2, U2.46 (SH_A)
- new net H2: U2.19 (INH_B)
- new net H2_LOW: U2.39 (SL_B)
- new net H2_VS: C28.2, R16.2, U2.41 (SH_B)
- new net H3: U2.21 (INH_C)
- new net H3_LOW: U2.34 (SL_C)
- new net H3_VS: C29.2, R14.2, U2.36 (SH_C)
- new net L1: U2.18 (INL_A)
- new net L2: U2.20 (INL_B)
- new net L3: U2.22 (INL_C)
- new net M_H1: U2.47 (GH_A)
- new net M_H2: U2.42 (GH_B)
- new net M_H3: U2.37 (GH_C)
- new net M_L1: U2.45 (GL_A)
- new net M_L2: U2.40 (GL_B)
- new net M_L3: U2.35 (GL_C)
- new net OC_ADJ: C18.1, C19.1, NT1.2, U2.11 (OC_ADJ)
- new net PH: C30.2, D8.1 (K), L1.1, U2.50 (PH), U2.51 (PH)
- new net RT_CLK: R9.2, U2.1 (RT_CLK)
- new net S1_N: U2.33 (SN1)
- new net S1_P: U2.32 (SP1)
- new net S2_N: U2.31 (SN2)
- new net S2_P: U2.30 (SP2)
- new net SENS1: R14.1, R15.2
- new net SENS2: R16.1, R17.2
- new net SENS3: R18.1, R19.2
- new net VSENSE: R12.1, R13.2, U2.3 (VSENSE)
- no-connect marks 0 -> 4
Other:
- note added: "BOOTSTRAP CAPS"
- note added: "BULK CAPACITOR KEEP AS CLOSE AS POSSIBLE TO THE IC AND TO THE DRIVER INPPUT LOOP"
- note added: "DECOUPLING CAPS PLACE AS CLOSE AS POSSIBLE TO THE IC"
- note added: "Hx_VS"
- note added: "INPUT PORTS"
- note added: "KEEP AWAY FROM NOISY TRACKS AND COMPONENTS"
- note added: "MCU SENSING FEEDBACK FOR EACH PHASE"
- note added: "OUTPUT PORTS"
- note added: "PHASE 1"
- note added: "PHASE 2"
- note added: "PHASE 3"
- note added: "SENSE 1 - PHASE 1"
- note added: "SENSE 2 - PHASE 2"
- note added: "[05] MOSFET DRIVER"
