File: Projects/AKK/BLDC_Motor_Controller/Design/rev01/rev01_1/Motor_Controller/[06] MOSFETS.kicad_sch (KiCad schematic)
At the start: 0 parts

Commit message: Update_03
Completed schematic.
Parts:
- added C48, C49: 2n2, symbol Device:C
- added J5, J6, J7: 7461084, symbol Connector_Generic:Conn_01x01
- added NT2, NT5, NT8: NetTie_2, symbol Device:NetTie_2
- added NT3, NT4, NT6, NT7, NT9: Net_Tie_PWR, symbol Device:NetTie_2
- added Q1, Q2, Q3, Q4, Q5, Q6: HSBA15810C, HSBA15810C_footprint_lib:PQFN-8_L6.0-W5.0-P1.27-LS6.0-BL, symbol HSBA15810C:HSBA15810C
- added R26, R27, R32, R33, R38, R39: 4R7, symbol Device:R
- added R28, R36, R42: 39K, symbol Device:R
- added R29, R30, R34, R35: 100R, symbol Device:R
- added R31, R37: 0R001, symbol Device:R
Connections:
- new net +VDC: Q1.5 (D), Q1.6 (D), Q1.7 (D), Q1.8 (D), Q1.9 (D), Q3.5 (D), Q3.6 (D), Q3.7 (D), Q3.8 (D), Q3.9 (D), Q5.5 (D), Q5.6 (D), Q5.7 (D), Q5.8 (D), Q5.9 (D)
- new net GND: NT4.1, NT7.1, NT9.1, R28.1, R36.1, R42.1
- new net H1_LOW: NT3.2, Q2.1 (S), Q2.2 (S), Q2.3 (S)
- new net H1_VS: NT2.1
- new net H2_LOW: NT6.2, Q4.1 (S), Q4.2 (S), Q4.3 (S)
- new net H2_VS: NT5.1
- new net H3_LOW: NT9.2, Q6.1 (S), Q6.2 (S), Q6.3 (S)
- new net H3_VS: NT8.1
- new net M_H1: R26.1
- new net M_H1_RG: Q1.4 (G), R26.2
- new net M_H2: R32.1
- new net M_H2_RG: Q3.4 (G), R32.2
- new net M_H3: R38.1
- new net M_H3_RG: Q5.4 (G), R38.2
- new net M_L1: R27.1
- new net M_L1_RG: Q2.4 (G), R27.2, R28.2
- new net M_L2: R33.1
- new net M_L2_RG: Q4.4 (G), R33.2, R36.2
- new net M_L3: R39.1
- new net M_L3_RG: Q6.4 (G), R39.2, R42.2
- new net PHASE_1: J5.1 (Pin_1), NT2.2, Q1.1 (S), Q1.2 (S), Q1.3 (S), Q2.5 (D), Q2.6 (D), Q2.7 (D), Q2.8 (D), Q2.9 (D)
- new net PHASE_2: J6.1 (Pin_1), NT5.2, Q3.1 (S), Q3.2 (S), Q3.3 (S), Q4.5 (D), Q4.6 (D), Q4.7 (D), Q4.8 (D), Q4.9 (D)
- new net PHASE_3: J7.1 (Pin_1), NT8.2, Q5.1 (S), Q5.2 (S), Q5.3 (S), Q6.5 (D), Q6.6 (D), Q6.7 (D), Q6.8 (D), Q6.9 (D)
- new net S1_N: C48.1, R29.1
- new net S1_P: C48.2, R30.1
- new net S2_N: C49.1, R34.1
- new net S2_P: C49.2, R35.1
- new net SH1_N: NT3.1, R29.2, R31.2
- new net SH1_P: NT4.2, R30.2, R31.1
- new net SH2_N: NT6.1, R34.2, R37.2
- new net SH2_P: NT7.2, R35.2, R37.1
Other:
- note added: "Hx_VS"
- note added: "MCU SENSING FEEDBACK FOR EACH PHASE"
- note added: "OUTPUT PHASE 1"
- note added: "OUTPUT PHASE 2"
- note added: "OUTPUT PHASE 3"
- note added: "PHASE 1"
- note added: "PHASE 2"
- note added: "PHASE 3"
- note added: "PLACE AS CLOSE AS POSSIBLE TO THE BULK CAPACITOR"
- note added: "Q_CONTROL"
- note added: "Q_SOURCES"
- note added: "ROUTE AS KELVING CONNECTIONS"
- note added: "SENSE 1"
- note added: "SENSE 2"
- note added: "[06] MOSFET"
