File: Projects/AKK/BLDC_Motor_Controller/Design/rev01/rev01_1/Motor_Controller/[07] CAN.kicad_sch (KiCad schematic)
At the start: 0 parts

Commit message: Update_03
Completed schematic.
Parts:
- added C50, C51: 51p, symbol Device:C
- added C52: 2u2, symbol Device:C
- added D15: ESDCAN24-2BLY, ESDCAN24-2BLY_footprint_lib:SOT-23-3_L3.0-W1.7-P0.95-LS2.9-BR, symbol ESDCAN24-2BLY:ESDCAN24-2BLY
- added FL1: 744227S, 744227S_footprint_lib:FILTER-SMD_4P-L9.2-W6.0-P2.54-TL, symbol Line_Filter:744227S
- added J8: Conn_01x04, Conn1x4_footprint_lib:CONN-SMD_S4B-XH-SM4-TB-LF-SN, symbol Conn_1x4:S4B-XH-SM4-TB-(LF)(SN)
- added R40: 120R, symbol Device:R
- added R41, R44: 10R, symbol Device:R
- added R43: 10k, symbol Device:R
- added U5: SN65HVD230, Package_SO:SOIC-8_3.9x4.9mm_P1.27mm, symbol Interface_CAN_LIN:SN65HVD230
Connections:
- new net: R43.2, U5.8 (Rs)
- new net +3V3: C52.1, U5.3 (VCC)
- new net +5V: J8.1
- new net CAN_N: FL1.4, U5.6 (CANL)
- new net CAN_P: FL1.3, U5.7 (CANH)
- new net CAN_RX: U5.4 (R)
- new net CAN_TX: U5.1 (D)
- new net C_CAN_N: C51.1, D15.2, J8.3, R40.2, R44.1
- new net C_CAN_P: C50.2, D15.1, J8.2, R40.1, R41.1
- new net GND: C50.1, C51.2, C52.2, D15.3, J8.4, R43.1, U5.2 (GND)
- new net R_CAN_N: FL1.1, R44.2
- new net R_CAN_P: FL1.2, R41.2
- no-connect marks 0 -> 3
Other:
- note added: "BYPASS CAP PLACE AS CLOSE AS POSIBLE TO THE IC"
- note added: "CAN_H AND CAN_L TO BE ROUTED AS DIFFERENTIAL PAIRS"
- note added: "MODE SELECTION RESISTOR SLEW RATE 0f-15 V/us MORE INFO IN DATASHEET"
- note added: "[07] CAN"
