File: Projects/AKK/BLDC_Motor_Controller/Design/rev01/rev01_1/Motor_Controller/[08] FILTERS.kicad_sch (KiCad schematic)
At the start: 0 parts

Commit message: Update_03
Completed schematic.
Parts:
- added C53, C56, C59, C60: 100n, symbol Device:C
- added C54, C55, C57, C58: 4n7, symbol Device:C
- added J6: Conn_01x06, Conn1x6_footprint_lib:CONN-SMD_S6B-XH-SM4-TB-LF-SN, symbol Conn_1x6:S6B-XH-SM4-TB(LF)(SN)
- added R45, R47, R49, R50: 2k2, symbol Device:R
- added R46, R48, R51, R52: 10k, symbol Device:R
Connections:
- new net +3V3: C53.1, C56.1, C59.1, C60.1, R45.1, R47.1, R49.1, R50.1
- new net +5V: J6.1
- new net GND: C53.2, C54.2, C55.2, C56.2, C57.2, C58.2, C59.2, C60.2, J6.6
- new net HALL_1_IN: C54.1, J6.3, R45.2, R46.1
- new net HALL_1_OUT: R46.2
- new net HALL_2_IN: C57.1, J6.4, R49.2, R51.1
- new net HALL_2_OUT: R51.2
- new net HALL_3_IN: C55.1, J6.5, R47.2, R48.1
- new net HALL_3_OUT: R48.2
- new net TEMP_IN: C58.1, J6.2, R50.2, R52.1
- new net TEMP_MOTOR: R52.2
- no-connect marks 0 -> 2
Other:
- note added: "HALL ENCODER INPUT"
- note added: "HALL ENCODER OUTPUT"
- note added: "HALL_1 FILTER"
- note added: "HALL_2 FILTER"
- note added: "HALL_3 FILTER"
- note added: "TEMP_MOTOR FILTER"
- note added: "TO MCU =>"
- note added: "[08] FILTERS"
