File: Projects/AKK/BLDC_Motor_Controller/Design/rev01/rev01_1/Motor_Controller/[09] USB.kicad_sch (KiCad schematic)
At the start: 0 parts

Commit message: Update_03
Completed schematic.
Parts:
- added J9: TYPE-C-31-M-12, symbol Connector:USB_C_Receptacle_USB2.0_16P
- added R53, R57, R59: 0R, symbol Device:R
- added R54, R55: 22R, symbol Device:R
- added R56, R58: 5k1, symbol Device:R
- added U6: PUSB3AB6Z, PUSB3AB6Z_footprint_lib:XSON-7_L2.2-W1.2-P0.50-BL, symbol PUSB3AB6Z:PUSB3AB6Z
Connections:
- new net: J9.S1 (SHIELD), R57.1, R59.1
- new net: J9.A4 (VBUS), J9.A9 (VBUS), J9.B4 (VBUS), J9.B9 (VBUS), R53.2
- new net +5V: R53.1
- new net +5V-C: U6.3 (CH2), U6.5 (CH4)
- new net CC1: J9.A5 (CC1), R58.1, U6.4 (CH3)
- new net CC2: J9.B5 (CC2), R56.1, U6.1 (CH1)
- new net GND: J9.A1 (GND), J9.A12 (GND), J9.B1 (GND), J9.B12 (GND), R56.2, R57.2, R58.2, R59.2, U6.2 (GND)
- new net USB-C_N: J9.A7 (D-), J9.B7 (D-), R54.1, U6.6 (CH5)
- new net USB-C_P: J9.A6 (D+), J9.B6 (D+), R55.1, U6.7 (CH6)
- new net USB_N: R54.2
- new net USB_P: R55.2
- no-connect marks 0 -> 2
Other:
- note added: "ESD PROTECTION PLACE AS CLOSE AS POSSIBLE TO THE CONNECTOR"
- note added: "FIT A 0R LINK, CAP OR RESISTOR"
- note added: "MOUNT A 0R JUMPER IF USED AS USB HOST"
- note added: "PULL-DOWN TELL THE HOT WE ARE UFP. ONLY ONE USED AT GIVEN TIME. BOTH NECESSARY FOR REVERSIBILITY."
- note added: "ROUTE AS DIFFERENTIAL PAIR"
- note added: "TERMINATING RESISTORS PLACE AS CLOSE AS POSSIBLE TO MCU"
- note added: "USB TO MCU"
- note added: "USB TYPE C ONLY 2.0"
- note added: "[09] USB"
