File: Projects/AKK/BLDC_Motor_Controller/Design/rev01/rev01_1/Motor_Controller/[10] MECHANICAL.kicad_sch (KiCad schematic)
At the start: 0 parts

Commit message: Update_03
Completed schematic.
Parts:
- added H1, H2, H3, H4: MountingHole_Pad, symbol Mechanical:MountingHole_Pad
- added R60, R61, R62, R63: 0R, symbol Device:R
Connections:
- new net: H4.1, R63.1
- new net: H3.1, R62.1
- new net: H1.1, R60.1
- new net: H2.1, R61.1
- new net GND: R60.2, R61.2, R62.2, R63.2
Other:
- note added: "- BOOT PIN PULLED-DOWN TO GND"
- note added: "- CHANGE PHASE SENSE RESISTORS"
- note added: "- CHANGED BULK CAPACITOR"
- note added: "- CHANGED NETS SENSE PHASES TO DIFFERENTIAL PAIRS"
- note added: "- INVERTED TX AND RX CONNECTOR PINS"
- note added: "- THERMISTOR MOVED TO LOWER LEG OF THE ADC PIN"
- note added: "BOARD NAME"
- note added: "BOARD NAME AND REVISION"
- note added: "B_NAME1 MOTOR_CONTROLLER_REV01_1"
- note added: "DF_LOGO"
- note added: "DF_LOGO_NO_SLK"
- note added: "DF_QR_CODE"
- note added: "FIT A ZERO OHM LINK, CAP, OR RESISTOR"
- note added: "L1"
- note added: "L2"
- note added: "L3"
- note added: "L4"
- note added: "LABELS"
- note added: "LOGO1 DF_LOGO"
- note added: "LOGO2 DF_LOGO_NO_SLK"
- note added: "LOGOS"
- note added: "M.DATE"
- note added: "MODIFICATION FROM VESC 4.11:"
- note added: "MOUNTING HOLES"
- note added: "M_DATE"
- note added: "M_DATE1 M_DATE"
- note added: "NOTES"
- note added: "NOTES1 NOTES"
- note added: "PCB"
- note added: "PCB1 PCB"
- note added: "QR1 DF_QR_CODE"
- note added: "[10] MECHANICAL"
